File: Barebones ATMega328P.sch (EAGLE design)
At the start: 3 parts, among them IC1 ATMEGA328P-AU

Commit message: v. 0.9
Parts:
- removed CN1: (no value), adafruit:DCBARRELPTH
- added 5V-CON, GND-CON, PWR-IN: PINHD-1X3, Connector:PINHD-1X3
- added C1, C2: 10uF, rcl:CPOL-EUE5-8.5
- added C3, C4: 22pF, rcl:C-EU025-025X050
- added C5: 1uF, rcl:CPOL-EUE5-8.5
- added IC2: 7805TV, linear:7805TV
- added JP1: PINHD-1X7, Connector:PINHD-1X7
- added JP2: PINHD-1X6, Connector:PINHD-1X6
- added LED1: RED, led:LED3MM
- added LED2: GREEN, led:LED3MM
- added Q1: (no value), adafruit:CRYSTALHC49S
- added R1: 220R, rcl:R-EU_0207/10
- added R2: 1K, rcl:R-EU_0207/10
- added R3: 10k, rcl:R-EU_0207/10
- added R4: 0R, rcl:R-EU_0207/10
- added SW1: 1-1825910-3, Switches:1-1825910-3
Connections:
- new net (PCINT10/ADC2)PC2: IC1G$1.(PCINT10/ADC2)PC2, JP1.4
- new net (PCINT11/ADC3)PC3: IC1G$1.(PCINT11/ADC3)PC3, JP1.5
- new net (PCINT12/SDA/ADC4)PC4: IC1G$1.(PCINT12/SDA/ADC4)PC4, JP1.6
- new net (PCINT13/SCL/ADC5)PC5: IC1G$1.(PCINT13/SCL/ADC5)PC5, JP1.7
- new net (PCINT8/ADC0)PC0: IC1G$1.(PCINT8/ADC0)PC0, JP1.2
- new net (PCINT9/ADC1)PC1: IC1G$1.(PCINT9/ADC1)PC1, JP1.3
- new net 10: IC1G$1.PD6(AIN0/OC0A/PCINT22), JP2.2
- new net 11: IC1G$1.PD7(AIN1/PCINT23), JP2.3
- new net 12: IC1G$1.(PCINT0/CLKO/ICP1)PB0, JP2.4
- new net 13: IC1G$1.(PCINT1/OC1A)PB1, JP2.5
- new net 14: IC1G$1.(PCINT2/OC1B/!SS!)PB2, JP2.6
- new net 9: IC1G$1.PD5(T1/OC0B/PCINT21), JP2.1
- new net ADC7: IC1G$1.ADC7, JP1.1
- new net GND: C1.-, C2.-, C3.1, C4.1, GND-CON.1, GND-CON.2, GND-CON.3, IC2.GND, ICSP.6, LED1.C, LED2.C, PWR-IN.3, SW1.1
- new net MISO: IC1G$1.(PCINT4/MISO)PB4, ICSP.1
- new net MOSI: IC1G$1.(PCINT3/OC2A/MOSI)PB3, ICSP.4
- new net N$1: LED1.A, R1.1
- new net N$2: R3.1, SW1.4
- new net N$3: C5.-, IC1G$1.PC6(!RESET!/PCINT14), SW1.3
- new net N$4: ICSP.2, R4.1
- new net N$5: LED2.A, R2.2
- new net PB6: C4.2, IC1G$1.PB6(XTAL1/TOSC1/PCINT6), Q1.2
- new net PB7: C3.2, IC1G$1.PB7(XTAL2/TOSC2/PCINT7), Q1.1
- new net RESET: C5.+, ICSP.5
- new net SCK: IC1G$1.(PCINT5/SCK)PB5, ICSP.3, R2.1
- new net VCC: 5V-CON.1, 5V-CON.2, 5V-CON.3, C2.+, IC1G$1.AVCC, IC2.VO, R1.2, R3.2, R4.2
- new net VIN: C1.+, IC2.VI, PWR-IN.1
Other:
- moved on the sheet: ICSP
